Commit message: Add husky model locally, add edited iris model to be moved to PX4 repo clone

File: models/urdf/husky.urdf.xacro (robot description, xacro)
@@ -43,10 +43,10 @@
   <xacro:arg name="urdf_extras" default="empty.urdf" />
   <!-- Included URDF/XACRO Files -->
-  <xacro:include filename="$(find husky_description)/urdf/decorations.urdf.xacro" />
-  <xacro:include filename="$(find husky_description)/urdf/wheel.urdf.xacro" />
-  <xacro:include filename="$(find husky_description)/urdf/accessories/intel_realsense.urdf.xacro"/>
-  <xacro:include filename="$(find husky_description)/urdf/accessories/sick_lms1xx_mount.urdf.xacro"/>
-  <xacro:include filename="$(find husky_description)/urdf/accessories/sensor_arch.urdf.xacro"/>
-  <xacro:include filename="$(find husky_description)/urdf/accessories/vlp16_mount.urdf.xacro"/>
+  <xacro:include filename="$(find mrs_uwb_sim)/models/urdf/decorations.urdf.xacro" />
+  <xacro:include filename="$(find mrs_uwb_sim)/models/urdf/wheel.urdf.xacro" />
+  <xacro:include filename="$(find mrs_uwb_sim)/models/urdf/accessories/intel_realsense.urdf.xacro"/>
+  <xacro:include filename="$(find mrs_uwb_sim)/models/urdf/accessories/sick_lms1xx_mount.urdf.xacro"/>
+  <xacro:include filename="$(find mrs_uwb_sim)/models/urdf/accessories/sensor_arch.urdf.xacro"/>
+  <xacro:include filename="$(find mrs_uwb_sim)/models/urdf/accessories/vlp16_mount.urdf.xacro"/>
   <xacro:property name="M_PI" value="3.14159"/>
   <!-- Base Size -->
@@ -66,5 +66,5 @@
       <origin xyz="0 0 0" rpy="0 0 0" />
       <geometry>
-        <mesh filename="package://husky_description/meshes/base_link.dae" />
+        <mesh filename="package://mrs_uwb_sim/models/meshes/base_link.dae" />
       </geometry>
     </visual>
