Commit message: fix mesh pats in additional xacro files

File: models/urdf/decorations.urdf.xacro (robot description, xacro)
@@ -39,5 +39,5 @@
         <origin xyz="0 0 0" rpy="0 0 0" />
         <geometry>
-          <mesh filename="package://husky_description/meshes/top_chassis.dae" />
+          <mesh filename="package://mrs_uwb_sim/models/meshes/top_chassis.dae" />
         </geometry>
       </visual>
@@ -53,5 +53,5 @@
         <visual>
           <geometry>
-            <mesh filename="package://husky_description/meshes/user_rail.dae" />
+            <mesh filename="package://mrs_uwb_sim/models/meshes/user_rail.dae" />
           </geometry>
         </visual>
@@ -69,5 +69,5 @@
         <visual>
           <geometry>
-            <mesh filename="package://husky_description/meshes/bumper.dae" />
+            <mesh filename="package://mrs_uwb_sim/models/meshes/bumper.dae" />
           </geometry>
         </visual>
@@ -83,5 +83,5 @@
             <visual>
                 <geometry>
-                    <mesh filename="package://husky_description/meshes/bumper_extension.dae" />
+                    <mesh filename="package://mrs_uwb_sim/models/meshes/bumper_extension.dae" />
                 </geometry>
             </visual>
@@ -99,5 +99,5 @@
         <visual>
           <geometry>
-            <mesh filename="package://husky_description/meshes/bumper.dae" />
+            <mesh filename="package://mrs_uwb_sim/models/meshes/bumper.dae" />
           </geometry>
         </visual>
@@ -113,5 +113,5 @@
             <visual>
                 <geometry>
-                    <mesh filename="package://husky_description/meshes/bumper_extension.dae" />
+                    <mesh filename="package://mrs_uwb_sim/models/meshes/bumper_extension.dae" />
                 </geometry>
             </visual>
@@ -131,5 +131,5 @@
             <origin xyz="0 0 0" rpy="0 0 0" />
             <geometry>
-              <mesh filename="package://husky_description/meshes/large_top_plate.dae" />
+              <mesh filename="package://mrs_uwb_sim/models/meshes/large_top_plate.dae" />
             </geometry>
           </visual>
@@ -137,5 +137,5 @@
             <origin xyz="0 0 0" rpy="0 0 0"/>
             <geometry>
-              <mesh filename="package://husky_description/meshes/large_top_plate_collision.stl" />
+              <mesh filename="package://mrs_uwb_sim/models/meshes/large_top_plate_collision.stl" />
             </geometry>
           </collision>
@@ -165,5 +165,5 @@
             <origin xyz="0 0 0" rpy="0 0 0" />
             <geometry>
-              <mesh filename="package://husky_description/meshes/top_plate.dae" />
+              <mesh filename="package://mrs_uwb_sim/models/meshes/top_plate.dae" />
             </geometry>
           </visual>
@@ -171,5 +171,5 @@
             <origin xyz="0 0 0" rpy="0 0 0"/>
             <geometry>
-              <mesh filename="package://husky_description/meshes/top_plate.stl" />
+              <mesh filename="package://mrs_uwb_sim/models/meshes/top_plate.stl" />
             </geometry>
           </collision>

File: models/urdf/wheel.urdf.xacro (robot description, xacro)
@@ -32,5 +32,5 @@
 				<origin xyz="0 0 0" rpy="0 0 0" />
 				<geometry>
-					<mesh filename="package://husky_description/meshes/wheel.dae" />
+					<mesh filename="package://mrs_uwb_sim/models/meshes/wheel.dae" />
 				</geometry>
 			</visual>
